Commit message: Update jackal.urdf.xacro

File: jackalpc/dvpg_jackal/urdf/jackal.urdf.xacro (robot description, xacro)
@@ -218,18 +218,4 @@
     <origin xyz="${mount_spacing} 0 0" />
   </joint>
-  <link name="velodyne">
-    <visual>
-      <origin xyz="0.0 0.0 0.0" />
-      <geometry>
-        <cylinder length="0.07" radius="0.05" />
-      </geometry>
-      <material name="gray" />
-    </visual>
-  </link>
-  <joint name="velodyne_joint" type="fixed">
-    <parent link="chassis_link" />
-    <child link="velodyne" />
-    <origin xyz="0.0 0.0 0.48" rpy="0 0 0" />
-  </joint>
   <!-- Bring in simulation data for Gazebo. -->
   <xacro:include filename="$(find jackal_description)/urdf/jackal.gazebo" />

Commit message: Update jackal.urdf.xacro

File: jackalpc/dvpg_jackal/urdf/jackal.urdf.xacro (robot description, xacro)
@@ -17,4 +17,6 @@
   <material name="yellow"><color rgba="0.8 0.8 0.0 1.0" /></material>
   <material name="black"><color rgba="0.15 0.15 0.15 1.0" /></material>
+  <material name="gray"><color rgba="0.2 0.2 0.2 1" /></material>
+  <material name="orange"><color rgba="1.0 0.5 0.2 1" /></material>
   <xacro:macro name="wheel" params="prefix *joint_pose">
     <link name="${prefix}_wheel_link">
@@ -185,4 +187,19 @@
     <child link="imu_link" />
   </joint>
+  <!-- external IMU Link -->
+  <link name="yahboom_link">
+    <visual>
+      <origin xyz="0.0 0.0 0.0" />
+      <geometry>
+        <box size="0.06 0.04 0.02" />
+      </geometry>
+      <material name="orange" />
+    </visual>
+  </link>
+  <joint name="yahboom_joint" type="fixed">
+    <parent link="chassis_link" />
+    <child link="yahboom_link" />
+    <origin xyz="0.0 0.0 0.1815" rpy="0 0 0" />
+  </joint>
   <!-- Default NAVSAT Link -->
   <link name="navsat_link">
@@ -217,4 +234,24 @@
     <child link="front_mount" />
     <origin xyz="${mount_spacing} 0 0" />
+  </joint>
+  <link name="velodyne">
+    <visual>
+      <origin xyz="0.0 0.0 0.0" />
+      <geometry>
+        <cylinder length="0.07" radius="0.05" />
+      </geometry>
+      <material name="gray" />
+    </visual>
+  </link>
+  <joint name="velodyne_joint" type="fixed">
+    <parent link="base_link" />
+    <child link="velodyne" />
+    <origin xyz="0.15 0.0 0.195" rpy="0 0 0" />
+  </joint>
+  <link name="front_laser"/>
+  <joint name="front_laser_joint" type="fixed">
+    <parent link="velodyne" />
+    <child link="front_laser" />
+    <origin xyz="0 0 0" rpy="0 0 0" />
   </joint>
   <!-- Bring in simulation data for Gazebo. -->

Commit message: Update jackal.urdf.xacro

File: jackalpc/dvpg_jackal/urdf/jackal.urdf.xacro (robot description, xacro)
@@ -217,4 +217,19 @@
     <origin xyz="-0.180 0.126 0.1815" />
   </joint>
+  <!-- Ex gps Link -->
+  <link name="gps">
+    <visual>
+      <geometry>
+        <cylinder radius="0.026" length="0.016" />
+      </geometry>
+      <origin xyz="0 0 0.008" />
+      <material name="black" />
+    </visual>
+  </link>
+  <joint name="gps_joint" type="fixed">
+    <parent link="chassis_link" />
+    <child link="gps" />
+    <origin xyz="-0.180 -0.126 0.1815" />
+  </joint>
   <link name="mid_mount"></link>
   <joint name="mid_mount_joint" type="fixed">
